File: T03_Schematic.sch (EAGLE design)
At the start: 25 parts, among them U1 ATMEGA328P-MU

Commit message: new schematic
Parts:
- removed G1: SL-340/SM3.6V, battery:SL-340/SM3.6V
- removed R8: (no value), adafruit:R-US_M0805
- removed U1: ATMEGA328P-MU, Ava:ATMEGA328P-MU
- added BAT1: (no value), SparkFun-Electromechanical:BATTERYAAA
- added HEADER: AVR_SPI_PRG_6PTH, SparkFun-Connectors:AVR_SPI_PRG_6PTH
- added U2: ATMEGA328P_PDIP, SparkFun-DigitalIC:ATMEGA328P_PDIP
Connections:
- new net N$11: HEADER.3, U2.PB5(SCK)
- new net N$12: HEADER.5, U2.PC6(/RESET)
- new net N$7: HEADER.4, U2.PB3(MOSI/OC2)
- new net N$8: HEADER.6, U2.GND@2
- new net N$9: HEADER.1, U2.PB4(MISO)
- net CATH1: now also U2.PD3(INT1); no longer U1.PD0
- net CATH2: now also U2.PD4(XCK/T0); no longer U1.PD1
- net CATH3: now also U2.PD5(T1); no longer U1.PD2
- net CATH4: no longer U1.PB3
- net CONTROL: no longer U1.PB4
- net GND: now also BAT1.-; no longer G1.+, R8.1, U1.ADC6, U1.ADC7, U1.AREF, U1.GND
- net GREN1: now also U2.PD6(AIN0); no longer U1.PD3
- net GREN2: now also U2.PD7(AIN1); no longer U1.PD4
- net GREN3: now also U2.PB0(ICP); no longer U1.PD5
- net PLAY1: no longer U1.PB1
- net PLAY2: no longer U1.PB2
- net RED1: now also U2.PD0(RXD); no longer U1.PD6
- net RED2: now also U2.PD1(TXD); no longer U1.PD7
- net RED3: now also U2.PD2(INT0); no longer U1.PB0
- net SELECT: no longer R8.2, U1.PB5
- net VCC: now also BAT1.+, U2.AVCC, U2.VCC; no longer G1.-, U1.AVCC, U1.VCC, U1.VCC_2
- net XTAL1: no longer U1.PB6
- net XTAL2: no longer U1.PB7
Other:
- note added: "1"
- moved on the sheet: BY1, BY2, BYCAP, CRYSTAL, LD1, LD10, LD2, LD3, LD4, LD5, LD6, LD7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

Commit message: new version
Parts:
- removed BAT1: (no value), SparkFun-Electromechanical:BATTERYAAA
- removed R5, R7: (no value), adafruit:R-US_M0805
- added BYCAP1, BYCAP2: 10u, adafruit:C-USC0805
- added INPINS: (no value), con-lsta:FE05-1
- added R8, R9: 1k, adafruit:R-US_M0805
- added TP1, TP10, TP11, TP12, TP13, TP14, TP15, TP16, TP17, TP18, TP19, TP2, TP20, TP21, TP22, TP23, TP24, TP3, TP4, TP5, TP6, TP7, TP8, TP9: PTR1B1,27, testpad:PTR1B1,27
- added VR: 317EMP, linear:317EMP
- BY1, BY2: value (none) -> 100n
- BYCAP: value (none) -> 10u
- CRYSTAL: value (none) -> 16MHz
- R1: value (none) -> 220
- R2, R3, R4: value (none) -> 330
- R6: value (none) -> 10k
- SELECT_BUTTON: value SPST_TACT-KMR2 -> SPST_TACT-EVQQ2; device adafruit:SPST_TACT-KMR2 -> adafruit:SPST_TACT-EVQQ2
Connections:
- removed net CONTROL: R7.1
- removed net N$4: R5.2
- removed net N$5: R7.2
- removed net N$7: HEADER.4, U2.PB3(MOSI/OC2)
- removed net N$9: HEADER.1, U2.PB4(MISO)
- removed net XTAL2: BY1.1, CRYSTAL.1
- new net AIN0: R9.1, U2.PC0(ADC0)
- new net N$13: BY1.1, CRYSTAL.1, TP22.TP, U2.PB7(XTAL2/TOSC2)
- new net SELECTPIN: INPINS.2, R9.2, TP15.TP
- new net V+POT: INPINS.3, R8.2, TP16.TP
- new net VIN: BYCAP2.1, INPINS.5, TP18.TP, VR.VI
- net CATH4: now also HEADER.4, U2.PB3(MOSI/OC2)
- net GND: now also BYCAP1.2, BYCAP2.2, INPINS.1, INPINS.4, TP14.TP, TP17.TP, VR.ADJ; no longer BAT1.-
- net GREN1: now also TP6.TP
- net GREN2: now also TP5.TP
- net GREN3: now also TP4.TP
- net N$1: now also TP7.TP
- net N$10: now also TP10.TP
- net N$3: now also TP8.TP
- net N$6: now also TP9.TP
- net N$8: now also TP24.TP, U2.GND@1
- net PLAY1: now also TP11.TP, U2.PB2(SS/OC1B)
- net PLAY2: now also HEADER.1, TP12.TP, U2.PB4(MISO)
- net RED1: now also TP1.TP
- net RED2: now also TP2.TP
- net RED3: now also TP3.TP
- net SELECT: now also TP20.TP, U2.PB1(OC1A)
- net VCC: now also BYCAP1.1, HEADER.2, R8.1, TP13.TP, TP19.TP, TP23.TP, U2.AREF, VR.VO; no longer BAT1.+, R5.1
- net XTAL1: now also TP21.TP, U2.PB6(XTAL1/TOSC1)
Other:
- note added: "6"
- note added: "Crystal resonator"
- note added: "External potentiometer through header pins"
- note added: "LED for player indicator"
- note added: "LED matrix for game-play"
- note added: "Programmer header pins"
- note added: "Pushbutton to select a move"
- note added: "Tic Tac Toe Game with LEDs"
- note added: "Voltage regulator through header pins from battery."
- note removed: "1"
- moved on the sheet: BYCAP, HEADER, LD1, LD10, LD2, LD3, LD4, LD5, LD6, LD7, LD8, LD9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
